Commit message: Move joint from multi_functional_servo_bracket_with_servo to outside of macro

File: src/strawberry_picking_rpi_description/urdf/multi_functional_servo_bracket_with_servo.urdf.xacro (robot description, xacro)
@@ -1,5 +1,5 @@
 <?xml version="1.0"?>
 <robot xmlns:xacro="http://www.ros.org/wiki/xacro" name="multi_functional_servo_bracket_with_servo">
-    <xacro:macro name="multi_functional_servo_bracket_with_servo" params="prefix parent_link *bracket_origin *joint_origin">
+    <xacro:macro name="multi_functional_servo_bracket_with_servo" params="prefix *bracket_origin *joint">
         <link name="${prefix}_multi_functional_servo_bracket_with_servo">
             <inertial>
@@ -33,9 +33,5 @@
             </collision>
         </link>
-        <joint name="${prefix}_multi_functional_servo_bracket_with_servo_to_${parent_link}" type="fixed">
-            <xacro:insert_block name="joint_origin"/>
-            <parent link="${parent_link}"/>
-            <child link="${prefix}_multi_functional_servo_bracket_with_servo"/>
-        </joint>
+        <xacro:insert_block name="joint"/>
     </xacro:macro>
 </robot>

Commit message: Add reverse mode for multi_functional_servo_bracket_with_servo.urdf.xacro because I wasn't aware that some servos are installed backwards

File: src/strawberry_picking_rpi_description/urdf/multi_functional_servo_bracket_with_servo.urdf.xacro (robot description, xacro)
@@ -1,5 +1,11 @@
 <?xml version="1.0"?>
 <robot xmlns:xacro="http://www.ros.org/wiki/xacro" name="multi_functional_servo_bracket_with_servo">
-    <xacro:macro name="multi_functional_servo_bracket_with_servo" params="prefix *bracket_origin *joint">
+    <xacro:macro name="multi_functional_servo_bracket_with_servo" params="prefix is_reversed:='false' *bracket_origin *joint">
+        <xacro:property name="reversed_servo">
+            <mesh filename="package://strawberry_picking_rpi_description/meshes/multi_functional_servo_bracket_with_servo_reverse.stl" scale="0.001 0.001 0.001"/>
+        </xacro:property>
+        <xacro:property name="normal_servo">
+            <mesh filename="package://strawberry_picking_rpi_description/meshes/multi_functional_servo_bracket_with_servo.stl" scale="0.001 0.001 0.001"/>
+        </xacro:property>
         <link name="${prefix}_multi_functional_servo_bracket_with_servo">
             <inertial>
@@ -11,18 +17,36 @@
                 <xacro:insert_block name="bracket_origin"/>
                 <geometry>
-                    <mesh filename="package://strawberry_picking_rpi_description/meshes/multi_functional_servo_bracket_with_servo.stl" scale="0.001 0.001 0.001"/>
+                    <xacro:if value="${is_reversed == 'true'}">
+                        <xacro:insert_block name="reversed_servo"/>
+                    </xacro:if>
+                    <xacro:if value="${is_reversed == 'false'}">
+                        <xacro:insert_block name="normal_servo"/>
+                    </xacro:if>
                 </geometry>
                 <material name="aluminum"/>
             </visual>
             <collision>
-                <origin xyz="
-                0.0
-                ${multi_functional_servo_bracket_with_servo_y_size/2}
-                0.013"
-                rpy="
-                0.0
-                0.0
-                0.0"
-                />
+                <xacro:if value="${is_reversed == 'true'}">
+                    <origin xyz="
+                    0.0
+                    ${-multi_functional_servo_bracket_with_servo_y_size/2}
+                    0.011"
+                    rpy="
+                    0.0
+                    0.0
+                    0.0"
+                    />
+                </xacro:if>
+                <xacro:if value="${is_reversed == 'false'}">
+                    <origin xyz="
+                    0.0
+                    ${multi_functional_servo_bracket_with_servo_y_size/2}
+                    0.011"
+                    rpy="
+                    0.0
+                    0.0
+                    0.0"
+                    />
+                </xacro:if>
                 <geometry>
                     <box size="${multi_functional_servo_bracket_with_servo_x_size}

Commit message: Replace multi_function_servo_bracket_with_servo stls with centered stls, adjust their urdfs

File: src/strawberry_picking_rpi_description/urdf/multi_functional_servo_bracket_with_servo.urdf.xacro (robot description, xacro)
@@ -27,26 +27,5 @@
             </visual>
             <collision>
-                <xacro:if value="${is_reversed == 'true'}">
-                    <origin xyz="
-                    0.0
-                    ${-multi_functional_servo_bracket_with_servo_y_size/2}
-                    0.011"
-                    rpy="
-                    0.0
-                    0.0
-                    0.0"
-                    />
-                </xacro:if>
-                <xacro:if value="${is_reversed == 'false'}">
-                    <origin xyz="
-                    0.0
-                    ${multi_functional_servo_bracket_with_servo_y_size/2}
-                    0.011"
-                    rpy="
-                    0.0
-                    0.0
-                    0.0"
-                    />
-                </xacro:if>
+                <xacro:insert_block name="bracket_origin"/>
                 <geometry>
                     <box size="${multi_functional_servo_bracket_with_servo_x_size}

Commit message: Redo servo brackets

File: src/strawberry_picking_rpi_description/urdf/multi_functional_servo_bracket_with_servo.urdf.xacro (robot description, xacro)
@@ -1,11 +1,11 @@
 <?xml version="1.0"?>
 <robot xmlns:xacro="http://www.ros.org/wiki/xacro" name="multi_functional_servo_bracket_with_servo">
+    <xacro:property name="servo">
+        <mesh filename="package://strawberry_picking_rpi_description/meshes/mg996r_servo.stl" scale="0.001 0.001 0.001"/>
+    </xacro:property>
+    <xacro:property name="servo_reversed">
+        <mesh filename="package://strawberry_picking_rpi_description/meshes/mg996r_servo_reversed.stl" scale="0.001 0.001 0.001"/>
+    </xacro:property>
     <xacro:macro name="multi_functional_servo_bracket_with_servo" params="prefix is_reversed:='false' *bracket_origin *joint">
-        <xacro:property name="reversed_servo">
-            <mesh filename="package://strawberry_picking_rpi_description/meshes/multi_functional_servo_bracket_with_servo_reverse.stl" scale="0.001 0.001 0.001"/>
-        </xacro:property>
-        <xacro:property name="normal_servo">
-            <mesh filename="package://strawberry_picking_rpi_description/meshes/multi_functional_servo_bracket_with_servo.stl" scale="0.001 0.001 0.001"/>
-        </xacro:property>
         <link name="${prefix}_multi_functional_servo_bracket_with_servo">
             <inertial>
@@ -17,10 +17,5 @@
                 <xacro:insert_block name="bracket_origin"/>
                 <geometry>
-                    <xacro:if value="${is_reversed == 'true'}">
-                        <xacro:insert_block name="reversed_servo"/>
-                    </xacro:if>
-                    <xacro:if value="${is_reversed == 'false'}">
-                        <xacro:insert_block name="normal_servo"/>
-                    </xacro:if>
+                    <mesh filename="package://strawberry_picking_rpi_description/meshes/multi_functional_servo_bracket.stl" scale="0.001 0.001 0.001"/>
                 </geometry>
                 <material name="aluminum"/>
@@ -36,4 +31,22 @@
             </collision>
         </link>
+        <link name="${prefix}_servo">
+            <visual>
+                <xacro:insert_block name="bracket_origin"/>
+                <geometry>
+                    <xacro:if value="${is_reversed == 'true'}">
+                        <xacro:insert_block name="servo_reversed"/>
+                    </xacro:if>
+                    <xacro:if value="${is_reversed == 'false'}">
+                        <xacro:insert_block name="servo"/>
+                    </xacro:if>
+                </geometry>
+                <material name="black_plastic"/>
+            </visual>
+        </link>
+        <joint name="${prefix}_servo_to_${prefix}_multi_functional_servo_bracket_with_servo" type="fixed">
+            <parent link="${prefix}_multi_functional_servo_bracket_with_servo"/>
+            <child link="${prefix}_servo"/>
+        </joint>
         <xacro:insert_block name="joint"/>
     </xacro:macro>

File: src/strawberry_picking_rpi_description/urdf/strawberry_picking_rpi.urdf.xacro (robot description, xacro)
@@ -28,4 +28,7 @@
         <color rgba="${136/255} ${139/255} ${141/255} 1.0"/>
     </material>
+    <material name="black_plastic">
+        <color rgba="${15/255} ${15/255} ${19/255} 1.0"/>
+    </material>
     <!-- the base link is the plank where the robot sits on -->
     <link name="base_link">
@@ -114,6 +117,6 @@
         <origin xyz="
         0.0
-        ${multi_functional_servo_bracket_with_servo_y_size/2}
-        0.011"
+        ${multi_functional_servo_bracket_with_servo_y_size/2+0.0008}
+        0.01"
         rpy="
         0.0
@@ -164,7 +167,7 @@
     <xacro:multi_functional_servo_bracket_with_servo prefix="2" is_reversed="true">
         <origin xyz="
-        0.001
-        ${-multi_functional_servo_bracket_with_servo_y_size/2}
-        0.0105"
+        0.0
+        ${-multi_functional_servo_bracket_with_servo_y_size/2-0.0015}
+        0.009"
         rpy="
         0.0
@@ -240,6 +243,6 @@
         <origin xyz="
         0.0095
-        -0.0015
-        ${-multi_functional_servo_bracket_with_servo_y_size}"
+        0.0
+        ${-multi_functional_servo_bracket_with_servo_y_size-0.003}"
         rpy="
         0.0
@@ -307,3 +310,54 @@
         </joint>
     </xacro:long_u_type_servo_bracket>
+    <!-- the next block will define the fourth segment of the robotic arm -->
+    <xacro:multi_functional_servo_bracket_with_servo prefix="4" is_reversed="false">
+        <origin xyz="
+        0.0095
+        0.0
+        ${-multi_functional_servo_bracket_with_servo_y_size}"
+        rpy="
+        0.0
+        0.0
+        0.0"
+        />
+        <joint name="4_multi_functional_servo_bracket_with_servo_to_4_long_u_type_servo_bracket" type="revolute">
+            <origin xyz="
+            ${-long_u_type_servo_bracket_y_size}
+            ${-long_u_type_servo_bracket_x_size+0.0025}
+            ${0.002}"
+            rpy="
+            ${pi}
+            ${pi/2}
+            0.0"
+            />
+            <limit lower="0" upper="${pi}" effort="1000" velocity="1.0"/>
+            <axis xyz="0.0 0.0 1"/>
+            <parent link="4_long_u_type_servo_bracket"/>
+            <child link="4_multi_functional_servo_bracket_with_servo"/>
+        </joint>
+    </xacro:multi_functional_servo_bracket_with_servo>
+    <xacro:multi_functional_servo_bracket_with_servo prefix="5" is_reversed="true">
+        <origin xyz="
+        0.007
+        ${multi_functional_servo_bracket_with_servo_y_size/2}
+        0.0"
+        rpy="
+        ${pi}
+        ${-pi/2}
+        0.0"
+        />
+        <joint name="5_multi_functional_servo_bracket_with_servo_to_4_multi_functional_servo_bracket_with_servo" type="fixed">
+            <origin xyz="
+            ${multi_functional_servo_bracket_with_servo_z_size/2-0.004}
+            ${multi_functional_servo_bracket_with_servo_y_size/2}
+            ${-multi_functional_servo_bracket_with_servo_z_size/2+0.003}"
+            rpy="
+            0.0
+            0.0
+            0.0"
+            />
+            <parent link="4_multi_functional_servo_bracket_with_servo"/>
+            <child link="5_multi_functional_servo_bracket_with_servo"/>
+        </joint>
+    </xacro:multi_functional_servo_bracket_with_servo>
 </robot>

Commit message: Modified multi functional servo bracket so that it renders properly in rviz2

File: src/strawberry_picking_rpi_description/urdf/multi_functional_servo_bracket_with_servo.urdf.xacro (robot description, xacro)
@@ -1,11 +1,5 @@
 <?xml version="1.0"?>
 <robot xmlns:xacro="http://www.ros.org/wiki/xacro" name="multi_functional_servo_bracket_with_servo">
-    <xacro:property name="servo">
-        <mesh filename="package://strawberry_picking_rpi_description/meshes/mg996r_servo.stl" scale="0.001 0.001 0.001"/>
-    </xacro:property>
-    <xacro:property name="servo_reversed">
-        <mesh filename="package://strawberry_picking_rpi_description/meshes/mg996r_servo_reversed.stl" scale="0.001 0.001 0.001"/>
-    </xacro:property>
-    <xacro:macro name="multi_functional_servo_bracket_with_servo" params="prefix is_reversed:='false' *bracket_origin *joint">
+    <xacro:macro name="multi_functional_servo_bracket_with_servo" params="prefix is_reversed:='' *bracket_origin *joint">
         <link name="${prefix}_multi_functional_servo_bracket_with_servo">
             <inertial>
@@ -35,10 +29,5 @@
                 <xacro:insert_block name="bracket_origin"/>
                 <geometry>
-                    <xacro:if value="${is_reversed == 'true'}">
-                        <xacro:insert_block name="servo_reversed"/>
-                    </xacro:if>
-                    <xacro:if value="${is_reversed == 'false'}">
-                        <xacro:insert_block name="servo"/>
-                    </xacro:if>
+                    <mesh filename="package://strawberry_picking_rpi_description/meshes/mg996r_servo${is_reversed}.stl" scale="0.001 0.001 0.001"/>
                 </geometry>
                 <material name="black_plastic"/>

File: src/strawberry_picking_rpi_description/urdf/strawberry_picking_rpi.urdf.xacro (robot description, xacro)
@@ -2,6 +2,6 @@
 <robot xmlns:xacro="http://www.ros.org/wiki/xacro" name="strawberry_picking_rpi">
     <!-- based on 2x2 plank measurements 1.5in x 1.5in x 1.5in -->
-    <xacro:property name="base_x_size" value="0.0381"/>
-    <xacro:property name="base_y_size" value="0.0381"/>
+    <xacro:property name="base_x_size" value="1.5"/>
+    <xacro:property name="base_y_size" value="4"/>
     <xacro:property name="base_z_size" value="0.0381"/>
     <xacro:property name="u_type_robot_waist_bracket_x_size" value="0.090"/>
@@ -114,5 +114,5 @@
         />
     </xacro:u_type_robot_waist_bracket>
-    <xacro:multi_functional_servo_bracket_with_servo prefix="1" is_reversed="false">
+    <xacro:multi_functional_servo_bracket_with_servo prefix="1">
         <origin xyz="
         0.0
@@ -165,5 +165,5 @@
         </joint>
     </xacro:long_u_type_servo_bracket>
-    <xacro:multi_functional_servo_bracket_with_servo prefix="2" is_reversed="true">
+    <xacro:multi_functional_servo_bracket_with_servo prefix="2" is_reversed="_reversed">
         <origin xyz="
         0.0
@@ -240,5 +240,5 @@
     </xacro:long_u_type_servo_bracket>
     <!-- the next blocks will define the third segment of the robotic arm -->
-    <xacro:multi_functional_servo_bracket_with_servo prefix="3" is_reversed="true">
+    <xacro:multi_functional_servo_bracket_with_servo prefix="3" is_reversed="_reversed">
         <origin xyz="
         0.0095
@@ -311,5 +311,5 @@
     </xacro:long_u_type_servo_bracket>
     <!-- the next block will define the fourth segment of the robotic arm -->
-    <xacro:multi_functional_servo_bracket_with_servo prefix="4" is_reversed="false">
+    <xacro:multi_functional_servo_bracket_with_servo prefix="4">
         <origin xyz="
         0.0095
@@ -337,5 +337,5 @@
         </joint>
     </xacro:multi_functional_servo_bracket_with_servo>
-    <xacro:multi_functional_servo_bracket_with_servo prefix="5" is_reversed="true">
+    <xacro:multi_functional_servo_bracket_with_servo prefix="5" is_reversed="_reversed">
         <origin xyz="
         0.007
