Commit message: Modify settings and continue development

File: src/strawberry_picking_rpi_description/urdf/strawberry_picking_rpi.urdf.xacro (robot description, xacro)
@@ -6,8 +6,12 @@
     <link name="base_link">
         <visual>
+            <origin xyz=" 0.0 0.0" rpy="0.0 0.0 0.0"/>
             <geometry>
                 <mesh filename="package://strawberry_picking_rpi_description/meshes/u_type_robot_waist_bracket.stl" scale="1.0"/>
             </geometry>
         </visual>
+        <collision>
+            <box size="$(base_x_size) $(base_y_size) $(base_z_size)"/>
+        </collision>
     </link>
 </robot>

Commit message: Save modifications

File: src/strawberry_picking_rpi_description/urdf/strawberry_picking_rpi.urdf.xacro (robot description, xacro)
@@ -12,5 +12,5 @@
         </visual>
         <collision>
-            <box size="$(base_x_size) $(base_y_size) $(base_z_size)"/>
+            <box size="${base_x_size} ${base_y_size} ${base_z_size}"/>
         </collision>
     </link>

Commit message: Create u_type_robot_waist_bracket.urdf.xacro

File: src/strawberry_picking_rpi_description/urdf/strawberry_picking_rpi.urdf.xacro (robot description, xacro)
@@ -1,17 +1,57 @@
 <?xml version="1.0"?>
-<robot name="strawberry_picking_rpi" xmlns:xacro="http://ros.org/wiki/xacro">
-    <xacro:property name="base_x_size" value="0.088" />
-    <xacro:property name="base_y_size" value="0.090" />
-    <xacro:property name="base_z_size" value="0.028" />
+<robot xmlns:xacro="http://www.ros.org/wiki/xacro" name="strawberry_picking_rpi">
+    <!-- based on 2x2 plank measurements 1.5in x 1.5in x 1.5in -->
+    <xacro:property name="base_x_size" value="0.0381"/>
+    <xacro:property name="base_y_size" value="0.0381"/>
+    <xacro:property name="base_z_size" value="0.0381"/>
+    <xacro:property name="u_type_robot_waist_bracket_x_size" value="0.090"/>
+    <xacro:property name="u_type_robot_waist_bracket_y_size" value="0.045"/>
+    <xacro:property name="u_type_robot_waist_bracket_z_size" value="0.028"/>
+    <xacro:include filename="$(find strawberry_picking_rpi_description)/urdf/u_type_robot_waist_bracket.urdf.xacro"/>
+    <material name="wood">
+        <color rgba="${164/255} ${116/255} ${73/255} 1.0"/>
+        <texture filename=""/>
+    </material>
+    <material name="aluminum">
+        <color rgba="${136/255} ${139/255} ${141/255} 1.0"/>
+        <texture filename="file_path"/>
+    </material>
     <link name="base_link">
-        <visual>
-            <origin xyz=" 0.0 0.0" rpy="0.0 0.0 0.0"/>
+        <inertial>
+            <origin xyz="0.0 0.0 ${u_type_robot_waist_bracket_z_size/2}" rpy="0.0 0.0 0.0"/>
+            <mass value="0.0"/>
+            <inertia ixx="0.0" ixy="0.0" ixz="0.0" iyy="0.0" iyz="0.0" izz="0.0"/>
+        </inertial>
+        <visual name="base_link">
+            <origin xyz="0.0 0.0 0.0" rpy="0.0 0.0 0.0"/>
             <geometry>
-                <mesh filename="package://strawberry_picking_rpi_description/meshes/u_type_robot_waist_bracket.stl" scale="1.0"/>
+                <box size="${base_x_size}
+                           ${base_y_size}
+                           ${base_z_size}"
+                />
             </geometry>
+            <material name="wood"/>
         </visual>
         <collision>
-            <box size="${base_x_size} ${base_y_size} ${base_z_size}"/>
+            <origin xyz="0.0 0.0 0.0" rpy="0.0 0.0 0.0"/>
+            <geometry>
+                <box size="${base_x_size}
+                           ${base_y_size}
+                           ${base_z_size}"
+                />
+            </geometry>
         </collision>
     </link>
+    <xacro:u_type_robot_waist_bracket prefix="01" parent_link="base_link">
+        <origin xyz=
+        "0.0
+        0.0
+        0.0"
+                rpy=
+        "0.0
+        0.0
+        0.0"
+        />
+        <origin xyz="0.0 0.0 ${base_z_size/2}" rpy="0.0 0.0 0.0"/>
+    </xacro:u_type_robot_waist_bracket>
 </robot>

Commit message: Create robot arm base

File: src/strawberry_picking_rpi_description/urdf/strawberry_picking_rpi.urdf.xacro (robot description, xacro)
@@ -2,6 +2,6 @@
 <robot xmlns:xacro="http://www.ros.org/wiki/xacro" name="strawberry_picking_rpi">
     <!-- based on 2x2 plank measurements 1.5in x 1.5in x 1.5in -->
-    <xacro:property name="base_x_size" value="0.0381"/>
-    <xacro:property name="base_y_size" value="0.0381"/>
+    <xacro:property name="base_x_size" value="0.25"/>
+    <xacro:property name="base_y_size" value="1"/>
     <xacro:property name="base_z_size" value="0.0381"/>
     <xacro:property name="u_type_robot_waist_bracket_x_size" value="0.090"/>
@@ -15,12 +15,7 @@
     <material name="aluminum">
         <color rgba="${136/255} ${139/255} ${141/255} 1.0"/>
-        <texture filename="file_path"/>
     </material>
+    <!-- the base link is the plank where the robot sits on -->
     <link name="base_link">
-        <inertial>
-            <origin xyz="0.0 0.0 ${u_type_robot_waist_bracket_z_size/2}" rpy="0.0 0.0 0.0"/>
-            <mass value="0.0"/>
-            <inertia ixx="0.0" ixy="0.0" ixz="0.0" iyy="0.0" iyz="0.0" izz="0.0"/>
-        </inertial>
         <visual name="base_link">
             <origin xyz="0.0 0.0 0.0" rpy="0.0 0.0 0.0"/>
@@ -43,15 +38,64 @@
         </collision>
     </link>
-    <xacro:u_type_robot_waist_bracket prefix="01" parent_link="base_link">
-        <origin xyz=
-        "0.0
+    <!-- these blocks define the base of the robotic arm -->
+    <xacro:u_type_robot_waist_bracket prefix="1" parent_link="base_link">
+        <origin xyz="
         0.0
-        0.0"
-                rpy=
-        "0.0
+        ${u_type_robot_waist_bracket_y_size/2}
+        ${u_type_robot_waist_bracket_z_size/2}"
+        rpy="
+        0.0
         0.0
         0.0"
         />
-        <origin xyz="0.0 0.0 ${base_z_size/2}" rpy="0.0 0.0 0.0"/>
+        <origin xyz="
+        0.0
+        0.0
+        ${base_z_size/2}"
+        rpy="
+        0.0
+        0.0
+        0.0"
+        />
+    </xacro:u_type_robot_waist_bracket>
+    <xacro:u_type_robot_waist_bracket prefix="2" parent_link="1_u_type_robot_waist_bracket">
+        <origin xyz="
+        0.0
+        ${-u_type_robot_waist_bracket_y_size/2}
+        ${u_type_robot_waist_bracket_z_size/2}"
+        rpy="
+        0.0
+        0.0
+        ${pi}"
+        />
+        <origin xyz="
+        0.0
+        0.0
+        0.0"
+        rpy="
+        0.0
+        0.0
+        0.0"
+        />
+    </xacro:u_type_robot_waist_bracket>
+    <xacro:u_type_robot_waist_bracket prefix="3" parent_link="1_u_type_robot_waist_bracket">
+        <origin xyz="
+        0.0
+        0.03025
+        ${u_type_robot_waist_bracket_z_size+u_type_robot_waist_bracket_y_size/2}"
+        rpy="
+        ${pi/2}
+        0.0
+        0.0"
+        />
+        <origin xyz="
+        0.0
+        0.0
+        0.0"
+        rpy="
+        0.0
+        0.0
+        0.0"
+        />
     </xacro:u_type_robot_waist_bracket>
 </robot>

Commit message: Added servo bracket with servo and fixed joint positions

File: src/strawberry_picking_rpi_description/urdf/strawberry_picking_rpi.urdf.xacro (robot description, xacro)
@@ -2,11 +2,15 @@
 <robot xmlns:xacro="http://www.ros.org/wiki/xacro" name="strawberry_picking_rpi">
     <!-- based on 2x2 plank measurements 1.5in x 1.5in x 1.5in -->
-    <xacro:property name="base_x_size" value="0.25"/>
-    <xacro:property name="base_y_size" value="1"/>
+    <xacro:property name="base_x_size" value="0.0381"/>
+    <xacro:property name="base_y_size" value="0.0381"/>
     <xacro:property name="base_z_size" value="0.0381"/>
     <xacro:property name="u_type_robot_waist_bracket_x_size" value="0.090"/>
     <xacro:property name="u_type_robot_waist_bracket_y_size" value="0.045"/>
     <xacro:property name="u_type_robot_waist_bracket_z_size" value="0.028"/>
+    <xacro:property name="multi_functional_servo_bracket_with_servo_x_size" value="0.057"/>
+    <xacro:property name="multi_functional_servo_bracket_with_servo_y_size" value="0.025"/>
+    <xacro:property name="multi_functional_servo_bracket_with_servo_z_size" value="0.050"/>
     <xacro:include filename="$(find strawberry_picking_rpi_description)/urdf/u_type_robot_waist_bracket.urdf.xacro"/>
+    <xacro:include filename="$(find strawberry_picking_rpi_description)/urdf/multi_functional_servo_bracket_with_servo.urdf.xacro"/>
     <material name="wood">
         <color rgba="${164/255} ${116/255} ${73/255} 1.0"/>
@@ -62,28 +66,8 @@
         <origin xyz="
         0.0
-        ${-u_type_robot_waist_bracket_y_size/2}
+        ${u_type_robot_waist_bracket_y_size/2}
         ${u_type_robot_waist_bracket_z_size/2}"
         rpy="
         0.0
-        0.0
-        ${pi}"
-        />
-        <origin xyz="
-        0.0
-        0.0
-        0.0"
-        rpy="
-        0.0
-        0.0
-        0.0"
-        />
-    </xacro:u_type_robot_waist_bracket>
-    <xacro:u_type_robot_waist_bracket prefix="3" parent_link="1_u_type_robot_waist_bracket">
-        <origin xyz="
-        0.0
-        0.03025
-        ${u_type_robot_waist_bracket_z_size+u_type_robot_waist_bracket_y_size/2}"
-        rpy="
-        ${pi/2}
         0.0
         0.0"
@@ -96,6 +80,46 @@
         0.0
         0.0
+        ${pi}"
+        />
+    </xacro:u_type_robot_waist_bracket>
+    <xacro:u_type_robot_waist_bracket prefix="3" parent_link="1_u_type_robot_waist_bracket">
+        <origin xyz="
+        0.0
+        0.0
+        ${u_type_robot_waist_bracket_y_size/2}"
+        rpy="
+        ${pi/2}
+        0.0
+        0.0"
+        />
+        <origin xyz="
+        0.0
+        0.03025
+        ${u_type_robot_waist_bracket_z_size}"
+        rpy="
+        0.0
+        0.0
         0.0"
         />
     </xacro:u_type_robot_waist_bracket>
+    <xacro:multi_functional_servo_bracket_with_servo prefix="1" parent_link="3_u_type_robot_waist_bracket">
+        <origin xyz="
+        0.0
+        0.0
+        0.0"
+        rpy="
+        0.0
+        0.0
+        0.0"
+        />
+        <origin xyz="
+        0.0
+        ${-u_type_robot_waist_bracket_z_size/2}
+        0.03025"
+        rpy="
+        0.0
+        0.0
+        ${pi}"
+        />
+    </xacro:multi_functional_servo_bracket_with_servo>
 </robot>

Commit message: Add first DOF :DD

File: src/strawberry_picking_rpi_description/urdf/strawberry_picking_rpi.urdf.xacro (robot description, xacro)
@@ -11,6 +11,10 @@
     <xacro:property name="multi_functional_servo_bracket_with_servo_y_size" value="0.025"/>
     <xacro:property name="multi_functional_servo_bracket_with_servo_z_size" value="0.050"/>
+    <xacro:property name="long_u_type_servo_bracket_x_size" value="0.055"/>
+    <xacro:property name="long_u_type_servo_bracket_y_size" value="0.025"/>
+    <xacro:property name="long_u_type_servo_bracket_z_size" value="0.065"/>
     <xacro:include filename="$(find strawberry_picking_rpi_description)/urdf/u_type_robot_waist_bracket.urdf.xacro"/>
     <xacro:include filename="$(find strawberry_picking_rpi_description)/urdf/multi_functional_servo_bracket_with_servo.urdf.xacro"/>
+    <xacro:include filename="$(find strawberry_picking_rpi_description)/urdf/long_u_type_servo_bracket.urdf.xacro"/>
     <material name="wood">
         <color rgba="${164/255} ${116/255} ${73/255} 1.0"/>
@@ -103,5 +107,5 @@
         />
     </xacro:u_type_robot_waist_bracket>
-    <xacro:multi_functional_servo_bracket_with_servo prefix="1" parent_link="3_u_type_robot_waist_bracket">
+    <xacro:multi_functional_servo_bracket_with_servo prefix="1">
         <origin xyz="
         0.0
@@ -113,13 +117,44 @@
         0.0"
         />
+        <joint name="1_multi_functional_servo_bracket_with_servo_to_3_u_type_robot_waist_bracket" type="fixed">
+            <origin xyz="
+            0.0
+            ${-u_type_robot_waist_bracket_z_size/2}
+            0.03025"
+            rpy="
+            0.0
+            0.0
+            ${pi}"
+            />
+            <parent link="3_u_type_robot_waist_bracket"/>
+            <child link="1_multi_functional_servo_bracket_with_servo"/>
+        </joint>
+    </xacro:multi_functional_servo_bracket_with_servo>
+    <!-- the next blocks will define the second segment of the robotic arm -->
+    <xacro:long_u_type_servo_bracket prefix="1">
         <origin xyz="
-        0.0
-        ${-u_type_robot_waist_bracket_z_size/2}
-        0.03025"
+        ${-long_u_type_servo_bracket_z_size+0.012}
+        ${-long_u_type_servo_bracket_y_size/2+0.002}
+        ${-long_u_type_servo_bracket_x_size/2+0.004}"
         rpy="
         0.0
-        0.0
-        ${pi}"
+        ${pi/2}
+        0.0"
         />
-    </xacro:multi_functional_servo_bracket_with_servo>
+        <joint name="1_long_u_type_servo_bracket_to_1_multi_functional_servo_bracket_with_servo" type="revolute">
+            <origin xyz="
+            0.010
+            ${multi_functional_servo_bracket_with_servo_y_size/2}
+            ${multi_functional_servo_bracket_with_servo_z_size-0.013}"
+            rpy="
+            0.0
+            0.0
+            ${-pi}"
+            />
+            <limit lower="0" upper="${pi}" effort="1000" velocity="1.0"/>
+            <axis xyz="0.0 0.0 1"/>
+            <parent link="1_multi_functional_servo_bracket_with_servo"/>
+            <child link="1_long_u_type_servo_bracket"/>
+        </joint>
+    </xacro:long_u_type_servo_bracket>
 </robot>

Commit message: Attach second servo

File: src/strawberry_picking_rpi_description/urdf/strawberry_picking_rpi.urdf.xacro (robot description, xacro)
@@ -107,5 +107,5 @@
         />
     </xacro:u_type_robot_waist_bracket>
-    <xacro:multi_functional_servo_bracket_with_servo prefix="1">
+    <xacro:multi_functional_servo_bracket_with_servo prefix="1" is_reversed="false">
         <origin xyz="
         0.0
@@ -136,5 +136,5 @@
         ${-long_u_type_servo_bracket_z_size+0.012}
         ${-long_u_type_servo_bracket_y_size/2+0.002}
-        ${-long_u_type_servo_bracket_x_size/2+0.004}"
+        ${-long_u_type_servo_bracket_x_size/2+0.002}"
         rpy="
         0.0
@@ -158,3 +158,27 @@
         </joint>
     </xacro:long_u_type_servo_bracket>
+    <xacro:multi_functional_servo_bracket_with_servo prefix="2" is_reversed="true">
+        <origin xyz="
+        0.0
+        0.0
+        0.0"
+        rpy="
+        0.0
+        0.0
+        0.0"
+        />
+        <joint name="2_multi_functional_servo_bracket_with_servo_to_1_long_u_type_servo_bracket" type="fixed">
+            <origin xyz="
+            -0.012
+            -0.011
+            0.003"
+            rpy="
+            ${pi/2}
+            ${pi}
+            ${pi}"
+            />
+            <parent link="1_long_u_type_servo_bracket"/>
+            <child link="2_multi_functional_servo_bracket_with_servo"/>
+        </joint>
+    </xacro:multi_functional_servo_bracket_with_servo>
 </robot>

Commit message: Create the third segment of the robotic arm

File: src/strawberry_picking_rpi_description/urdf/strawberry_picking_rpi.urdf.xacro (robot description, xacro)
@@ -110,10 +110,10 @@
         <origin xyz="
         0.0
-        0.0
-        0.0"
-        rpy="
-        0.0
-        0.0
-        0.0"
+        ${multi_functional_servo_bracket_with_servo_y_size/2}
+        0.011"
+        rpy="
+        0.0
+        0.0
+        ${pi}"
         />
         <joint name="1_multi_functional_servo_bracket_with_servo_to_3_u_type_robot_waist_bracket" type="fixed">
@@ -134,6 +134,6 @@
     <xacro:long_u_type_servo_bracket prefix="1">
         <origin xyz="
-        ${-long_u_type_servo_bracket_z_size+0.012}
-        ${-long_u_type_servo_bracket_y_size/2+0.002}
+        ${-long_u_type_servo_bracket_z_size+0.0125}
+        ${-long_u_type_servo_bracket_y_size/2+0.0025}
         ${-long_u_type_servo_bracket_x_size/2+0.002}"
         rpy="
@@ -144,7 +144,7 @@
         <joint name="1_long_u_type_servo_bracket_to_1_multi_functional_servo_bracket_with_servo" type="revolute">
             <origin xyz="
-            0.010
-            ${multi_functional_servo_bracket_with_servo_y_size/2}
-            ${multi_functional_servo_bracket_with_servo_z_size-0.013}"
+            0.0095
+            ${multi_functional_servo_bracket_with_servo_y_size/2+0.0015}
+            ${multi_functional_servo_bracket_with_servo_z_size-0.014}"
             rpy="
             0.0
@@ -160,7 +160,7 @@
     <xacro:multi_functional_servo_bracket_with_servo prefix="2" is_reversed="true">
         <origin xyz="
-        0.0
-        0.0
-        0.0"
+        0.001
+        ${-multi_functional_servo_bracket_with_servo_y_size/2}
+        0.0105"
         rpy="
         0.0
@@ -182,3 +182,79 @@
         </joint>
     </xacro:multi_functional_servo_bracket_with_servo>
+    <xacro:long_u_type_servo_bracket prefix="2">
+        <origin xyz="
+        ${-long_u_type_servo_bracket_z_size+0.0125}
+        ${-long_u_type_servo_bracket_y_size/2+0.0025}
+        ${-long_u_type_servo_bracket_x_size/2+0.001}"
+        rpy="
+        0.0
+        ${pi/2}
+        0.0"
+        />
+        <joint name="2_long_u_type_servo_bracket_to_2_multi_functional_servo_bracket_with_servo" type="revolute">
+            <origin xyz="
+            0.0095
+            ${-multi_functional_servo_bracket_with_servo_y_size/2-0.0015}
+            ${multi_functional_servo_bracket_with_servo_z_size-0.014}"
+            rpy="
+            0.0
+            0.0
+            0.0"
+            />
+            <limit lower="0" upper="${pi}" effort="1000" velocity="1.0"/>
+            <axis xyz="0.0 0.0 1"/>
+            <parent link="2_multi_functional_servo_bracket_with_servo"/>
+            <child link="2_long_u_type_servo_bracket"/>
+        </joint>
+    </xacro:long_u_type_servo_bracket>
+    <xacro:long_u_type_servo_bracket prefix="3">
+        <origin xyz="
+        ${-long_u_type_servo_bracket_z_size+0.012}
+        ${-long_u_type_servo_bracket_y_size/2+0.002}
+        ${-long_u_type_servo_bracket_x_size/2+0.002}"
+        rpy="
+        0.0
+        ${-pi/2}
+        0.0"
+        />
+        <joint name="3_long_u_type_servo_bracket_to_2_long_u_type_servo_bracket" type="fixed">
+            <origin xyz="
+            0.0
+            0.0
+            0.0"
+            rpy="
+            0.0
+            0.0
+            0.0"
+            />
+            <parent link="2_long_u_type_servo_bracket"/>
+            <child link="3_long_u_type_servo_bracket"/>
+        </joint>
+    </xacro:long_u_type_servo_bracket>
+    <xacro:multi_functional_servo_bracket_with_servo prefix="3" is_reversed="true">
+        <origin xyz="
+        0.0095
+        -0.0015
+        ${-multi_functional_servo_bracket_with_servo_y_size}"
+        rpy="
+        0.0
+        0.0
+        ${pi}"
+        />
+        <joint name="3_multi_functional_servo_bracket_with_servo_to_3_long_u_type_servo_bracket" type="revolute">
+            <origin xyz="
+            ${-long_u_type_servo_bracket_x_size*2+0.0045}
+            0.0
+            0.0"
+            rpy="
+            0.0
+            0.0
+            ${pi}"
+            />
+            <limit lower="0" upper="${pi}" effort="1000" velocity="1.0"/>
+            <axis xyz="0.0 0.0 1"/>
+            <parent link="3_long_u_type_servo_bracket"/>
+            <child link="3_multi_functional_servo_bracket_with_servo"/>
+        </joint>
+    </xacro:multi_functional_servo_bracket_with_servo>
 </robot>

Commit message: Apply the l_type_servo_bracket

File: src/strawberry_picking_rpi_description/urdf/strawberry_picking_rpi.urdf.xacro (robot description, xacro)
@@ -14,7 +14,11 @@
     <xacro:property name="long_u_type_servo_bracket_y_size" value="0.025"/>
     <xacro:property name="long_u_type_servo_bracket_z_size" value="0.065"/>
+    <xacro:property name="l_type_servo_bracket_x_size" value="0.037"/>
+    <xacro:property name="l_type_servo_bracket_y_size" value="0.025"/>
+    <xacro:property name="l_type_servo_bracket_z_size" value="0.025"/>
     <xacro:include filename="$(find strawberry_picking_rpi_description)/urdf/u_type_robot_waist_bracket.urdf.xacro"/>
     <xacro:include filename="$(find strawberry_picking_rpi_description)/urdf/multi_functional_servo_bracket_with_servo.urdf.xacro"/>
     <xacro:include filename="$(find strawberry_picking_rpi_description)/urdf/long_u_type_servo_bracket.urdf.xacro"/>
+    <xacro:include filename="$(find strawberry_picking_rpi_description)/urdf/l_type_servo_bracket.urdf.xacro"/>
     <material name="wood">
         <color rgba="${164/255} ${116/255} ${73/255} 1.0"/>
@@ -259,3 +263,47 @@
         </joint>
     </xacro:multi_functional_servo_bracket_with_servo>
+    <xacro:l_type_servo_bracket prefix="1" parent_link="3_multi_functional_servo_bracket_with_servo">
+        <origin xyz="
+        0.0
+        -0.0062
+        ${l_type_servo_bracket_z_size/2-0.002}"
+        rpy="
+        0.0
+        0.0
+        0.0"
+        />
+        <origin xyz="
+        0.0205
+        ${-multi_functional_servo_bracket_with_servo_y_size/2-0.001}
+        ${-multi_functional_servo_bracket_with_servo_z_size/2}"
+        rpy="
+        ${3*pi/2}
+        ${pi/2}
+        0.0"
+        />
+    </xacro:l_type_servo_bracket>
+    <xacro:long_u_type_servo_bracket prefix="4">
+        <origin xyz="
+        0.0
+        0.0
+        ${-long_u_type_servo_bracket_y_size/2+0.0045}"
+        rpy="
+        ${pi/2}
+        0.0
+        0.0"
+        />
+        <joint name="4_long_u_type_servo_bracket_to_1_l_type_servo_bracket" type="fixed">
+            <origin xyz="
+            0.0
+            ${-l_type_servo_bracket_y_size}
+            ${l_type_servo_bracket_z_size/2}"
+            rpy="
+            0.0
+            0.0
+            0.0"
+            />
+            <parent link="1_l_type_servo_bracket"/>
+            <child link="4_long_u_type_servo_bracket"/>
+        </joint>
+    </xacro:long_u_type_servo_bracket>
 </robot>
