Commit message: Set mg996r velocity

File: src/strawberry_picking_rpi_description/urdf/strawberry_picking_rpi.urdf.xacro (robot description, xacro)
@@ -11,4 +11,5 @@
     <xacro:property name="multi_functional_servo_bracket_with_servo_y_size" value="0.025"/>
     <xacro:property name="multi_functional_servo_bracket_with_servo_z_size" value="0.050"/>
+    <xacro:property name="mg996r_velocity_6v" value="6.98133333333"/>
     <xacro:property name="long_u_type_servo_bracket_x_size" value="0.055"/>
     <xacro:property name="long_u_type_servo_bracket_y_size" value="0.025"/>
@@ -159,5 +160,5 @@
             ${-pi}"
             />
-            <limit lower="0" upper="${pi}" effort="1000" velocity="1.0"/>
+            <limit lower="0" upper="${pi}" effort="1000" velocity="${mg996r_velocity_6v}"/>
             <axis xyz="0.0 0.0 1"/>
             <parent link="1_multi_functional_servo_bracket_with_servo"/>
@@ -209,5 +210,5 @@
             0.0"
             />
-            <limit lower="0" upper="${pi}" effort="1000" velocity="1.0"/>
+            <limit lower="0" upper="${pi}" effort="1000" velocity="${mg996r_velocity_6v}"/>
             <axis xyz="0.0 0.0 1"/>
             <parent link="2_multi_functional_servo_bracket_with_servo"/>
@@ -260,5 +261,5 @@
             ${pi/2}"
             />
-            <limit lower="0" upper="${pi}" effort="1000" velocity="1.0"/>
+            <limit lower="0" upper="${pi}" effort="1000" velocity="${mg996r_velocity_6v}"/>
             <axis xyz="0.0 0.0 1"/>
             <parent link="3_long_u_type_servo_bracket"/>
@@ -331,5 +332,5 @@
             0.0"
             />
-            <limit lower="0" upper="${pi}" effort="1000" velocity="1.0"/>
+            <limit lower="0" upper="${pi}" effort="1000" velocity="${mg996r_velocity_6v}"/>
             <axis xyz="0.0 0.0 1"/>
             <parent link="4_long_u_type_servo_bracket"/>

Commit message: Set mg996r velocity 4.8v

File: src/strawberry_picking_rpi_description/urdf/strawberry_picking_rpi.urdf.xacro (robot description, xacro)
@@ -12,4 +12,5 @@
     <xacro:property name="multi_functional_servo_bracket_with_servo_z_size" value="0.050"/>
     <xacro:property name="mg996r_velocity_6v" value="6.98133333333"/>
+    <xacro:property name="mg996r_velocity_4.8v" value="5.51157894737"/>
     <xacro:property name="long_u_type_servo_bracket_x_size" value="0.055"/>
     <xacro:property name="long_u_type_servo_bracket_y_size" value="0.025"/>

Commit message: replace . with dot

File: src/strawberry_picking_rpi_description/urdf/strawberry_picking_rpi.urdf.xacro (robot description, xacro)
@@ -12,5 +12,5 @@
     <xacro:property name="multi_functional_servo_bracket_with_servo_z_size" value="0.050"/>
     <xacro:property name="mg996r_velocity_6v" value="6.98133333333"/>
-    <xacro:property name="mg996r_velocity_4.8v" value="5.51157894737"/>
+    <xacro:property name="mg996r_velocity_4dot8v" value="5.51157894737"/>
     <xacro:property name="long_u_type_servo_bracket_x_size" value="0.055"/>
     <xacro:property name="long_u_type_servo_bracket_y_size" value="0.025"/>

Commit message: Create arm control hardware interface package based on Example 1 of ros2 control demos

File: src/strawberry_picking_rpi_description/urdf/strawberry_picking_rpi.urdf.xacro (robot description, xacro)
@@ -376,3 +376,4 @@
     <!-- ros2_control part -->
     <xacro:include filename="$(find strawberry_picking_rpi_description)/urdf/strawberry_picking_rpi_control.urdf.xacro"/>
+    <xacro:controllers/>
 </robot>

File: src/strawberry_picking_rpi_description/urdf/strawberry_picking_rpi_control.urdf.xacro (robot description, xacro)
@@ -1,61 +1,49 @@
 <?xml version="1.0"?>
 <robot xmlns:xacro="http://www.ros.org/wiki/xacro" name="strawberry_picking_rpi_control">
-    <ros2_control name="robot_6_dof" type="system">
-        <hardware>
-            <plugin>
-                joint_trajectory_controller/JointTrajectoryController
-            </plugin>
-        </hardware>
-        <joint name="DOF_1">
-            <command_interface name="position">
-                <param name="min">0</param>
-                <param name="max">{pi}</param>
-            </command_interface>
-            <state_interface name="position"/>
-        </joint>
-        <joint name="DOF_2">
-            <command_interface name="position">
-                <param name="min">0</param>
-                <param name="max">{pi}</param>
-            </command_interface>
-            <state_interface name="position"/>
-        </joint>
-        <joint name="DOF_3">
-            <command_interface name="position">
-                <param name="min">0</param>
-                <param name="max">{pi}</param>
-            </command_interface>
-            <state_interface name="position"/>
-        </joint>
-        <joint name="DOF_4">
-            <command_interface name="position">
-                <param name="min">0</param>
-                <param name="max">{pi}</param>
-            </command_interface>
-            <state_interface name="position"/>
-        </joint>
-        <joint name="DOF_5">
-            <command_interface name="position">
-                <param name="min">0</param>
-                <param name="max">{pi}</param>
-            </command_interface>
-            <state_interface name="position"/>
-        </joint>
-        <!-- additional joints ...-->
-        <!-- additional hardware/sensors ...-->
-    </ros2_control>
-    <ros2_control name="gripper_controller" type="actuator">
-        <hardware>
-            <plugin>
-                position_controllers/GrippperActionController
-            </plugin>
-        </hardware>
-        <joint name="GRIPPER">
-            <command_interface name="position">
-                <param name="min">0</param>
-                <param name="max">1.1</param>
-            </command_interface>
-            <state_interface name="position"/>
-        </joint>
-    </ros2_control>
+    <xacro:macro name="controllers">
+        <ros2_control name="arm_controller" type="system">
+            <hardware>
+                <plugin>sprpi_arm_hwi/ArmHardwareInterface</plugin>
+                <param name="baud_rate">230400</param>
+                <param name="serial_port">/dev/ttyACM0</param>
+            </hardware>
+            <joint name="DOF_1">
+                <command_interface name="position">
+                    <param name="min">0</param>
+                    <param name="max">3.141519</param>
+                </command_interface>
+                <state_interface name="position"/>
+            </joint>
+            <joint name="DOF_2">
+                <command_interface name="position">
+                    <param name="min">0</param>
+                    <param name="max">3.141519</param>
+                </command_interface>
+                <state_interface name="position"/>
+            </joint>
+            <joint name="DOF_3">
+                <command_interface name="position">
+                    <param name="min">0</param>
+                    <param name="max">3.141519</param>
+                </command_interface>
+                <state_interface name="position"/>
+            </joint>
+            <joint name="DOF_4">
+                <command_interface name="position">
+                    <param name="min">0</param>
+                    <param name="max">3.141519</param>
+                </command_interface>
+                <state_interface name="position"/>
+            </joint>
+            <joint name="DOF_5">
+                <command_interface name="position">
+                    <param name="min">0</param>
+                    <param name="max">3.141519</param>
+                </command_interface>
+                <state_interface name="position"/>
+            </joint>
+            <!-- additional joints ...-->
+            <!-- additional hardware/sensors ...-->
+        </ros2_control>
+    </xacro:macro>
 </robot>

Commit message: Create the robotic base (kabaong) with baskets and mirrors in the urdf

File: src/strawberry_picking_rpi_description/urdf/strawberry_picking_rpi.urdf.xacro (robot description, xacro)
@@ -2,7 +2,7 @@
 <robot xmlns:xacro="http://www.ros.org/wiki/xacro" name="strawberry_picking_rpi">
     <!-- based on 2x2 plank measurements 1.5in x 1.5in x 1.5in -->
-    <xacro:property name="base_x_size" value="0.0381"/>
-    <xacro:property name="base_y_size" value="0.0381"/>
-    <xacro:property name="base_z_size" value="0.0381"/>
+    <xacro:property name="base_x_size" value="0.1"/>
+    <xacro:property name="base_y_size" value="0.1"/>
+    <xacro:property name="base_z_size" value="0.02"/>
     <xacro:property name="u_type_robot_waist_bracket_x_size" value="0.090"/>
     <xacro:property name="u_type_robot_waist_bracket_y_size" value="0.045"/>
@@ -24,4 +24,5 @@
     <xacro:include filename="$(find strawberry_picking_rpi_description)/urdf/l_type_servo_bracket.urdf.xacro"/>
     <xacro:include filename="$(find strawberry_picking_rpi_description)/urdf/gripper.urdf.xacro"/>
+    <xacro:include filename="$(find strawberry_picking_rpi_description)/urdf/robotic_base_with_accessories.urdf.xacro"/>
     <material name="wood">
         <color rgba="${164/255} ${116/255} ${73/255} 1.0"/>
@@ -377,3 +378,24 @@
     <!--<xacro:include filename="$(find strawberry_picking_rpi_description)/urdf/strawberry_picking_rpi_control.urdf.xacro"/>
     <xacro:controllers/>-->
+    <!-- the next block will define the robotic base with it's accessories (e.g. cameras) -->
+    <xacro:robotic_base_with_accessories parent_link="base_link">
+        <origin xyz="
+        0.0
+        0.0
+        0.0"
+        rpy="
+        0.0
+        0.0
+        0.0"
+        />
+        <origin xyz="
+        0.0
+        ${(base_y_size/2-kabaong_y_size/2)}
+        ${-(base_z_size/2+kabaong_z_size/2)}"
+        rpy="
+        0.0
+        0.0
+        0.0"
+        />
+    </xacro:robotic_base_with_accessories>
 </robot>
