Commit message: Apply gripper xacro to main file

File: src/strawberry_picking_rpi_description/urdf/gripper.urdf.xacro (robot description, xacro)
@@ -1,5 +1,5 @@
 <?xml version="1.0"?>
 <robot xmlns:xacro="http://www.ros.org/wiki/xacro" name="gripper">
-    <xacro:macro name="gripper" params="prefix">
+    <xacro:macro name="gripper" params="prefix *joint">
         <link name="gripper_base">
             <inertial>
@@ -228,6 +228,5 @@
             <origin xyz="0.002 -0.015 0.0305" rpy="0.0 0 0"/>
         </joint>
+        <xacro:insert_block name="joint"/>
     </xacro:macro>
-    <xacro:gripper prefix="1">
-    </xacro:gripper>
 </robot>

File: src/strawberry_picking_rpi_description/urdf/strawberry_picking_rpi.urdf.xacro (robot description, xacro)
@@ -2,6 +2,6 @@
 <robot xmlns:xacro="http://www.ros.org/wiki/xacro" name="strawberry_picking_rpi">
     <!-- based on 2x2 plank measurements 1.5in x 1.5in x 1.5in -->
-    <xacro:property name="base_x_size" value="1.5"/>
-    <xacro:property name="base_y_size" value="4"/>
+    <xacro:property name="base_x_size" value="0.0381"/>
+    <xacro:property name="base_y_size" value="0.0381"/>
     <xacro:property name="base_z_size" value="0.0381"/>
     <xacro:property name="u_type_robot_waist_bracket_x_size" value="0.090"/>
@@ -23,4 +23,5 @@
     <xacro:include filename="$(find strawberry_picking_rpi_description)/urdf/long_u_type_servo_bracket.urdf.xacro"/>
     <xacro:include filename="$(find strawberry_picking_rpi_description)/urdf/l_type_servo_bracket.urdf.xacro"/>
+    <xacro:include filename="$(find strawberry_picking_rpi_description)/urdf/gripper.urdf.xacro"/>
     <material name="wood">
         <color rgba="${164/255} ${116/255} ${73/255} 1.0"/>
@@ -363,3 +364,13 @@
         </joint>
     </xacro:multi_functional_servo_bracket_with_servo>
+    <xacro:gripper prefix="1">
+        <joint name="gripper_base_to_5_multi_functional_servo_bracket_with_servo" type="revolute">
+            <parent link="5_multi_functional_servo_bracket_with_servo"/>
+            <child link="gripper_base"/>
+            <origin xyz="0.034 0.012 0.01" rpy="${pi/2} 0.0 ${pi/2}"/>
+            <axis xyz="0.0 0.0 1"/>
+            <limit lower="0" upper="${pi}" effort="1000" velocity="${mg996r_velocity_6v}"/>
+            <axis xyz="0.0 0.0 1"/>
+        </joint>
+    </xacro:gripper>
 </robot>

Commit message: Add collision to the servo attached to the servo

File: src/strawberry_picking_rpi_description/urdf/gripper.urdf.xacro (robot description, xacro)
@@ -222,4 +222,10 @@
                 <material name="aluminum"/>
             </visual>
+            <collision>
+                <origin xyz="0.0275 -0.0095 0.0" rpy="${pi/2} ${pi} ${-pi/2}"/>
+                <geometry>
+                    <mesh filename="package://strawberry_picking_rpi_description/meshes/mg996r_servo_reversed.stl" scale="0.001 0.001 0.001"/>
+                </geometry>
+            </collision>
         </link>
         <joint name="gripper_servo_to_gripper_base" type="fixed">

Commit message: Rename DOFs and Gripper joints into more appropriate names

File: src/strawberry_picking_rpi_description/urdf/gripper.urdf.xacro (robot description, xacro)
@@ -36,5 +36,5 @@
             </visual>
         </link>
-        <joint name="gripper_palm_to_finger_large_lo_to_gripper_base" type="revolute">
+        <joint name="GRIPPER" type="revolute">
             <parent link="gripper_base"/>
             <child link="gripper_palm_to_finger_large_lo"/>
@@ -60,5 +60,5 @@
             <parent link="gripper_base"/>
             <child link="gripper_palm_to_finger_large"/>
-            <mimic joint="gripper_palm_to_finger_large_lo_to_gripper_base" multiplier="-1"/>
+            <mimic joint="GRIPPER" multiplier="-1"/>
             <axis xyz="1 0 0"/>
             <limit lower="-3.14159" upper="3.14159" velocity="50.0" effort="1000.0"/>
@@ -83,5 +83,5 @@
             <child link="gripper_palm_to_finger_small_left_over"/>
             <axis xyz="1 0 0"/>
-            <mimic joint="gripper_palm_to_finger_large_lo_to_gripper_base" multiplier="-1"/>
+            <mimic joint="GRIPPER" multiplier="-1"/>
             <limit lower="-3.14159" upper="3.14159" velocity="50.0" effort="1000.0"/>
             <origin xyz="0.0 0.0068 0.052" rpy="0 0 0"/>
@@ -105,5 +105,5 @@
             <child link="gripper_palm_to_finger_small_left_under"/>
             <axis xyz="1 0 0"/>
-            <mimic joint="gripper_palm_to_finger_large_lo_to_gripper_base" multiplier="-1"/>
+            <mimic joint="GRIPPER" multiplier="-1"/>
             <limit lower="-3.14159" upper="3.14159" velocity="50.0" effort="1000.0"/>
             <origin xyz="0.004 0.0068 0.052" rpy="0 0 0"/>
@@ -127,5 +127,5 @@
             <child link="gripper_palm_to_finger_small_right_over"/>
             <axis xyz="1 0 0"/>
-            <mimic joint="gripper_palm_to_finger_large_lo_to_gripper_base"/>
+            <mimic joint="GRIPPER"/>
             <limit lower="-3.14159" upper="3.14159" velocity="50.0" effort="1000.0"/>
             <origin xyz="0.0 -0.0068 0.052" rpy="0 0 0"/>
@@ -149,5 +149,5 @@
             <child link="gripper_palm_to_finger_small_right_under"/>
             <axis xyz="1 0 0"/>
-            <mimic joint="gripper_palm_to_finger_large_lo_to_gripper_base"/>
+            <mimic joint="GRIPPER"/>
             <limit lower="-3.14159" upper="3.14159" velocity="50.0" effort="1000.0"/>
             <origin xyz="0.004 -0.0068 0.052" rpy="0 0 0"/>

File: src/strawberry_picking_rpi_description/urdf/strawberry_picking_rpi.urdf.xacro (robot description, xacro)
@@ -152,5 +152,5 @@
         0.0"
         />
-        <joint name="1_long_u_type_servo_bracket_to_1_multi_functional_servo_bracket_with_servo" type="revolute">
+        <joint name="DOF_1" type="revolute">
             <origin xyz="
             0.0095
@@ -202,5 +202,5 @@
         0.0"
         />
-        <joint name="2_long_u_type_servo_bracket_to_2_multi_functional_servo_bracket_with_servo" type="revolute">
+        <joint name="DOF_2" type="revolute">
             <origin xyz="
             0.0095
@@ -253,5 +253,5 @@
         ${pi}"
         />
-        <joint name="3_multi_functional_servo_bracket_with_servo_to_3_long_u_type_servo_bracket" type="revolute">
+        <joint name="DOF_3" type="revolute">
             <origin xyz="
             ${-long_u_type_servo_bracket_x_size*2+0.0045}
@@ -324,5 +324,5 @@
         0.0"
         />
-        <joint name="4_multi_functional_servo_bracket_with_servo_to_4_long_u_type_servo_bracket" type="revolute">
+        <joint name="DOF_4" type="revolute">
             <origin xyz="
             ${-long_u_type_servo_bracket_y_size}
@@ -365,5 +365,5 @@
     </xacro:multi_functional_servo_bracket_with_servo>
     <xacro:gripper prefix="1">
-        <joint name="gripper_base_to_5_multi_functional_servo_bracket_with_servo" type="revolute">
+        <joint name="DOF_5" type="revolute">
             <parent link="5_multi_functional_servo_bracket_with_servo"/>
             <child link="gripper_base"/>

Commit message: Fix inversed (i uninversed it) control for gripper

File: src/strawberry_picking_rpi_description/urdf/gripper.urdf.xacro (robot description, xacro)
@@ -24,10 +24,10 @@
         <link name="gripper_palm_to_finger_large_lo">
             <inertial>
-                <origin xyz="0.0 0.0 0.0" rpy="${pi/2} ${pi} ${pi/2}"/>
-                <mass value="0.0"/>
-                <inertia ixx="0.0" ixy="0.0" ixz="0.0" iyy="0.0" iyz="0.0" izz="0.0"/>
-            </inertial>
-            <visual>
-                <origin xyz="-0.00075 0.0 0.0" rpy="${pi/2} ${pi} ${pi/2}"/>
+                <origin xyz="0.0 0.0 0.0" rpy="${pi/2} ${pi-1.1} ${pi/2}"/>
+                <mass value="0.0"/>
+                <inertia ixx="0.0" ixy="0.0" ixz="0.0" iyy="0.0" iyz="0.0" izz="0.0"/>
+            </inertial>
+            <visual>
+                <origin xyz="-0.00075 0.0 0.0" rpy="${pi/2} ${pi-1.1} ${pi/2}"/>
                 <geometry>
                     <mesh filename="package://strawberry_picking_rpi_description/meshes/gripper_palm_to_finger_large_lo.stl" scale="0.001 0.001 0.001"/>
@@ -39,5 +39,5 @@
             <parent link="gripper_base"/>
             <child link="gripper_palm_to_finger_large_lo"/>
-            <axis xyz="1 0 0"/>
+            <axis xyz="-1 0 0"/>
             <limit lower="0.0" upper="1.1" velocity="50.0" effort="1000.0"/>
             <origin xyz="-0.002 -0.015 0.03" rpy="0 0 0"/>
@@ -45,10 +45,10 @@
         <link name="gripper_palm_to_finger_large">
             <inertial>
-                <origin xyz="0.0 0.0 0.0" rpy="${pi/2} ${pi} ${pi/2}"/>
-                <mass value="0.0"/>
-                <inertia ixx="0.0" ixy="0.0" ixz="0.0" iyy="0.0" iyz="0.0" izz="0.0"/>
-            </inertial>
-            <visual>
-                <origin xyz="-0.00075 0.0 0.0" rpy="${pi/2} ${pi} ${-pi/2}"/>
+                <origin xyz="0.0 0.0 0.0" rpy="${pi/2} ${pi-1.1} ${pi/2}"/>
+                <mass value="0.0"/>
+                <inertia ixx="0.0" ixy="0.0" ixz="0.0" iyy="0.0" iyz="0.0" izz="0.0"/>
+            </inertial>
+            <visual>
+                <origin xyz="-0.00075 0.0 0.0" rpy="${pi/2} ${pi-1.1} ${-pi/2}"/>
                 <geometry>
                     <mesh filename="package://strawberry_picking_rpi_description/meshes/gripper_palm_to_finger_large.stl" scale="0.001 0.001 0.001"/>
@@ -60,94 +60,94 @@
             <parent link="gripper_base"/>
             <child link="gripper_palm_to_finger_large"/>
+            <mimic joint="GRIPPER"/>
+            <axis xyz="1 0 0"/>
+            <limit lower="-3.14159" upper="3.14159" velocity="50.0" effort="1000.0"/>
+            <origin xyz="0.0 0.012 0.03" rpy="0 0 0"/>
+        </joint>
+        <link name="gripper_palm_to_finger_small_left_over">
+            <inertial>
+                <origin xyz="0.0 0.0 0.0" rpy="${pi/2} ${pi-1.1} ${pi/2}"/>
+                <mass value="0.0"/>
+                <inertia ixx="0.0" ixy="0.0" ixz="0.0" iyy="0.0" iyz="0.0" izz="0.0"/>
+            </inertial>
+            <visual>
+                <origin xyz="-0.00075 0.0 0.0" rpy="${pi/2} ${pi-1.1} ${-pi/2}"/>
+                <geometry>
+                    <mesh filename="package://strawberry_picking_rpi_description/meshes/gripper_palm_to_finger_small.stl" scale="0.001 0.001 0.001"/>
+                </geometry>
+                <material name="aluminum"/>
+            </visual>
+        </link>
+        <joint name="gripper_palm_to_finger_small_left_over_to_gripper_base" type="revolute">
+            <parent link="gripper_base"/>
+            <child link="gripper_palm_to_finger_small_left_over"/>
+            <axis xyz="1 0 0"/>
+            <mimic joint="GRIPPER"/>
+            <limit lower="-3.14159" upper="3.14159" velocity="50.0" effort="1000.0"/>
+            <origin xyz="0.0 0.0068 0.052" rpy="0 0 0"/>
+        </joint>
+        <link name="gripper_palm_to_finger_small_left_under">
+            <inertial>
+                <origin xyz="0.0 0.0 0.0" rpy="${pi/2} ${pi-1.1} ${pi/2}"/>
+                <mass value="0.0"/>
+                <inertia ixx="0.0" ixy="0.0" ixz="0.0" iyy="0.0" iyz="0.0" izz="0.0"/>
+            </inertial>
+            <visual>
+                <origin xyz="-0.00075 0.0 0.0" rpy="${pi/2} ${pi-1.1} ${-pi/2}"/>
+                <geometry>
+                    <mesh filename="package://strawberry_picking_rpi_description/meshes/gripper_palm_to_finger_small.stl" scale="0.001 0.001 0.001"/>
+                </geometry>
+                <material name="aluminum"/>
+            </visual>
+        </link>
+        <joint name="gripper_palm_to_finger_small_left_under_to_gripper_base" type="revolute">
+            <parent link="gripper_base"/>
+            <child link="gripper_palm_to_finger_small_left_under"/>
+            <axis xyz="1 0 0"/>
+            <mimic joint="GRIPPER"/>
+            <limit lower="-3.14159" upper="3.14159" velocity="50.0" effort="1000.0"/>
+            <origin xyz="0.004 0.0068 0.052" rpy="0 0 0"/>
+        </joint>
+        <link name="gripper_palm_to_finger_small_right_over">
+            <inertial>
+                <origin xyz="0.0 0.0 0.0" rpy="${pi/2} ${pi+1.1} ${pi/2}"/>
+                <mass value="0.0"/>
+                <inertia ixx="0.0" ixy="0.0" ixz="0.0" iyy="0.0" iyz="0.0" izz="0.0"/>
+            </inertial>
+            <visual>
+                <origin xyz="-0.00075 0.0 0.0" rpy="${pi/2} ${pi+1.1} ${-pi/2}"/>
+                <geometry>
+                    <mesh filename="package://strawberry_picking_rpi_description/meshes/gripper_palm_to_finger_small.stl" scale="0.001 0.001 0.001"/>
+                </geometry>
+                <material name="aluminum"/>
+            </visual>
+        </link>
+        <joint name="gripper_palm_to_finger_small_right_over_to_gripper_base" type="revolute">
+            <parent link="gripper_base"/>
+            <child link="gripper_palm_to_finger_small_right_over"/>
+            <axis xyz="1 0 0"/>
             <mimic joint="GRIPPER" multiplier="-1"/>
-            <axis xyz="1 0 0"/>
-            <limit lower="-3.14159" upper="3.14159" velocity="50.0" effort="1000.0"/>
-            <origin xyz="0.0 0.012 0.03" rpy="0 0 0"/>
-        </joint>
-        <link name="gripper_palm_to_finger_small_left_over">
-            <inertial>
-                <origin xyz="0.0 0.0 0.0" rpy="${pi/2} ${pi} ${pi/2}"/>
-                <mass value="0.0"/>
-                <inertia ixx="0.0" ixy="0.0" ixz="0.0" iyy="0.0" iyz="0.0" izz="0.0"/>
-            </inertial>
-            <visual>
-                <origin xyz="-0.00075 0.0 0.0" rpy="${pi/2} ${pi} ${-pi/2}"/>
-                <geometry>
-                    <mesh filename="package://strawberry_picking_rpi_description/meshes/gripper_palm_to_finger_small.stl" scale="0.001 0.001 0.001"/>
-                </geometry>
-                <material name="aluminum"/>
-            </visual>
-        </link>
-        <joint name="gripper_palm_to_finger_small_left_over_to_gripper_base" type="revolute">
-            <parent link="gripper_base"/>
-            <child link="gripper_palm_to_finger_small_left_over"/>
+            <limit lower="-3.14159" upper="3.14159" velocity="50.0" effort="1000.0"/>
+            <origin xyz="0.0 -0.0068 0.052" rpy="0 0 0"/>
+        </joint>
+        <link name="gripper_palm_to_finger_small_right_under">
+            <inertial>
+                <origin xyz="0.0 0.0 0.0" rpy="${pi/2} ${pi+1.1} ${pi/2}"/>
+                <mass value="0.0"/>
+                <inertia ixx="0.0" ixy="0.0" ixz="0.0" iyy="0.0" iyz="0.0" izz="0.0"/>
+            </inertial>
+            <visual>
+                <origin xyz="-0.00075 0.0 0.0" rpy="${pi/2} ${pi+1.1} ${-pi/2}"/>
+                <geometry>
+                    <mesh filename="package://strawberry_picking_rpi_description/meshes/gripper_palm_to_finger_small.stl" scale="0.001 0.001 0.001"/>
+                </geometry>
+                <material name="aluminum"/>
+            </visual>
+        </link>
+        <joint name="gripper_palm_to_finger_small_right_under_to_gripper_base" type="revolute">
+            <parent link="gripper_base"/>
+            <child link="gripper_palm_to_finger_small_right_under"/>
             <axis xyz="1 0 0"/>
             <mimic joint="GRIPPER" multiplier="-1"/>
-            <limit lower="-3.14159" upper="3.14159" velocity="50.0" effort="1000.0"/>
-            <origin xyz="0.0 0.0068 0.052" rpy="0 0 0"/>
-        </joint>
-        <link name="gripper_palm_to_finger_small_left_under">
-            <inertial>
-                <origin xyz="0.0 0.0 0.0" rpy="${pi/2} ${pi} ${pi/2}"/>
-                <mass value="0.0"/>
-                <inertia ixx="0.0" ixy="0.0" ixz="0.0" iyy="0.0" iyz="0.0" izz="0.0"/>
-            </inertial>
-            <visual>
-                <origin xyz="-0.00075 0.0 0.0" rpy="${pi/2} ${pi} ${-pi/2}"/>
-                <geometry>
-                    <mesh filename="package://strawberry_picking_rpi_description/meshes/gripper_palm_to_finger_small.stl" scale="0.001 0.001 0.001"/>
-                </geometry>
-                <material name="aluminum"/>
-            </visual>
-        </link>
-        <joint name="gripper_palm_to_finger_small_left_under_to_gripper_base" type="revolute">
-            <parent link="gripper_base"/>
-            <child link="gripper_palm_to_finger_small_left_under"/>
-            <axis xyz="1 0 0"/>
-            <mimic joint="GRIPPER" multiplier="-1"/>
-            <limit lower="-3.14159" upper="3.14159" velocity="50.0" effort="1000.0"/>
-            <origin xyz="0.004 0.0068 0.052" rpy="0 0 0"/>
-        </joint>
-        <link name="gripper_palm_to_finger_small_right_over">
-            <inertial>
-                <origin xyz="0.0 0.0 0.0" rpy="${pi/2} ${pi} ${pi/2}"/>
-                <mass value="0.0"/>
-                <inertia ixx="0.0" ixy="0.0" ixz="0.0" iyy="0.0" iyz="0.0" izz="0.0"/>
-            </inertial>
-            <visual>
-                <origin xyz="-0.00075 0.0 0.0" rpy="${pi/2} ${pi} ${-pi/2}"/>
-                <geometry>
-                    <mesh filename="package://strawberry_picking_rpi_description/meshes/gripper_palm_to_finger_small.stl" scale="0.001 0.001 0.001"/>
-                </geometry>
-                <material name="aluminum"/>
-            </visual>
-        </link>
-        <joint name="gripper_palm_to_finger_small_right_over_to_gripper_base" type="revolute">
-            <parent link="gripper_base"/>
-            <child link="gripper_palm_to_finger_small_right_over"/>
-            <axis xyz="1 0 0"/>
-            <mimic joint="GRIPPER"/>
-            <limit lower="-3.14159" upper="3.14159" velocity="50.0" effort="1000.0"/>
-            <origin xyz="0.0 -0.0068 0.052" rpy="0 0 0"/>
-        </joint>
-        <link name="gripper_palm_to_finger_small_right_under">
-            <inertial>
-                <origin xyz="0.0 0.0 0.0" rpy="${pi/2} ${pi} ${pi/2}"/>
-                <mass value="0.0"/>
-                <inertia ixx="0.0" ixy="0.0" ixz="0.0" iyy="0.0" iyz="0.0" izz="0.0"/>
-            </inertial>
-            <visual>
-                <origin xyz="-0.00075 0.0 0.0" rpy="${pi/2} ${pi} ${-pi/2}"/>
-                <geometry>
-                    <mesh filename="package://strawberry_picking_rpi_description/meshes/gripper_palm_to_finger_small.stl" scale="0.001 0.001 0.001"/>
-                </geometry>
-                <material name="aluminum"/>
-            </visual>
-        </link>
-        <joint name="gripper_palm_to_finger_small_right_under_to_gripper_base" type="revolute">
-            <parent link="gripper_base"/>
-            <child link="gripper_palm_to_finger_small_right_under"/>
-            <axis xyz="1 0 0"/>
-            <mimic joint="GRIPPER"/>
             <limit lower="-3.14159" upper="3.14159" velocity="50.0" effort="1000.0"/>
             <origin xyz="0.004 -0.0068 0.052" rpy="0 0 0"/>
@@ -179,5 +179,5 @@
             <mimic joint="gripper_palm_to_finger_large_to_gripper_base" multiplier="-1"/>
             <limit lower="-3.14159" upper="3.14159" velocity="50.0" effort="1000.0"/>
-            <origin xyz="0.002 0.0 0.0305" rpy="0.34 0 0"/>
+            <origin xyz="0.002 0.0275 0.01425" rpy="0.34 0 0"/>
         </joint>
         <link name="finger_right">
@@ -207,5 +207,5 @@
             <mimic joint="gripper_palm_to_finger_large_to_gripper_base"/>
             <limit lower="-3.14159" upper="3.14159" velocity="50.0" effort="1000.0"/>
-            <origin xyz="0.002 0.0 0.0305" rpy="-0.38 0 0"/>
+            <origin xyz="0.002 -0.0275 0.01425" rpy="-0.38 0 0"/>
         </joint>
         <link name="gripper_servo">

File: src/strawberry_picking_rpi_description/urdf/model_for_moveit.urdf (robot description, URDF)
Before this commit: robot strawberry_picking_rpi, 34 links, 33 joints
Joints:
- joint GRIPPER: axis 1 0 0 -> -1 0 0
- joint finger_left_to_gripper_palm_to_finger_large: origin xyz=0.002 0.0 0.0305 rpy=0.34 0 0 -> xyz=0.002 0.0275 0.01425 rpy=0.34 0 0
- joint finger_right_to_gripper_palm_to_finger_large: origin xyz=0.002 0.0 0.0305 rpy=-0.38 0 0 -> xyz=0.002 -0.0275 0.01425 rpy=-0.38 0 0
- joint gripper_palm_to_finger_large_to_gripper_base: mimic joint=GRIPPER multiplier=-1 -> joint=GRIPPER
- joint gripper_palm_to_finger_small_left_over_to_gripper_base: mimic joint=GRIPPER multiplier=-1 -> joint=GRIPPER
- joint gripper_palm_to_finger_small_left_under_to_gripper_base: mimic joint=GRIPPER multiplier=-1 -> joint=GRIPPER
- joint gripper_palm_to_finger_small_right_over_to_gripper_base: mimic joint=GRIPPER -> joint=GRIPPER multiplier=-1
- joint gripper_palm_to_finger_small_right_under_to_gripper_base: mimic joint=GRIPPER -> joint=GRIPPER multiplier=-1
