Commit message: Fix rotation issues

File: src/strawberry_picking_rpi_description/urdf/model_for_moveit.urdf (robot description, URDF)
Before this commit: robot strawberry_picking_rpi, 29 links, 28 joints
Joints:
- joint DOF_3: axis 0.0 0.0 1 -> 0.0 0.0 -1; origin xyz=             -0.1055             0.0             0.0 rpy=             0.0             0.0             1.5707963267948966 -> xyz=             -0.1055             0.0             0.0 rpy=             0.0             0.0             -1.5707963267948966
- joint DOF_4: axis 0.0 0.0 1 -> 0.0 0.0 -1; origin xyz=             -0.025             -0.0525             0.002 rpy=             3.141592653589793             1.5707963267948966             0.0 -> xyz=             -0.025             -0.0525             0.002 rpy=             0.0             -1.5707963267948966             0.0

File: src/strawberry_picking_rpi_description/urdf/strawberry_picking_rpi.urdf.xacro (robot description, xacro)
@@ -261,8 +261,8 @@
             0.0
             0.0
-            ${pi/2}"
-            />
-            <limit lower="0" upper="${pi}" effort="1000" velocity="${mg996r_velocity_6v}"/>
-            <axis xyz="0.0 0.0 1"/>
+            ${-pi/2}"
+            />
+            <limit lower="0" upper="${pi}" effort="1000" velocity="${mg996r_velocity_6v}"/>
+            <axis xyz="0.0 0.0 -1"/>
             <parent link="3_long_u_type_servo_bracket"/>
             <child link="3_multi_functional_servo_bracket_with_servo"/>
@@ -330,10 +330,10 @@
             ${0.002}"
             rpy="
-            ${pi}
-            ${pi/2}
-            0.0"
-            />
-            <limit lower="0" upper="${pi}" effort="1000" velocity="${mg996r_velocity_6v}"/>
-            <axis xyz="0.0 0.0 1"/>
+            0.0
+            ${-pi/2}
+            0.0"
+            />
+            <limit lower="0" upper="${pi}" effort="1000" velocity="${mg996r_velocity_6v}"/>
+            <axis xyz="0.0 0.0 -1"/>
             <parent link="4_long_u_type_servo_bracket"/>
             <child link="4_multi_functional_servo_bracket_with_servo"/>
@@ -374,5 +374,5 @@
         </joint>
     </xacro:gripper>
-    <!-- ros2_control part, commented out for moveit2 -->
+    <!-- ros2_control part, commented out for MoveIt2 -->
     <!--<xacro:include filename="$(find strawberry_picking_rpi_description)/urdf/strawberry_picking_rpi_control.urdf.xacro"/>
     <xacro:controllers/>-->

Commit message: Update model used for moveit

File: src/strawberry_picking_rpi_description/urdf/model_for_moveit.urdf (robot description, URDF)
Before this commit: robot strawberry_picking_rpi, 29 links, 28 joints
Links:
- added link basket_diseased, mass 0.0; collision cylinder length=0.13 radius=0.085; visual cylinder length=0.13 radius=0.085
- added link basket_healthy, mass 0.0; collision cylinder length=0.13 radius=0.085; visual cylinder length=0.13 radius=0.085
- added link kabaong, mass 0.0; collision box size=0.85 0.25 0.05; visual box size=0.85 0.25 0.05
- added link mirror_left, mass 0.0; collision box size=0.03 0.105 0.15; visual box size=0.03 0.105 0.15
- added link mirror_right, mass 0.0; collision box size=0.03 0.105 0.15; visual box size=0.03 0.105 0.15
- link base_link: geometry collision box size=0.1 0.1 0.02; visual box size=0.1 0.1 0.02
Joints:
- added joint basket_diseased_to_kabaong: type fixed, parent kabaong, child basket_diseased, origin xyz=             -0.36              0.0              0.025 rpy=             0.0              0.0             0.0
- added joint basket_healthy_to_kabaong: type fixed, parent kabaong, child basket_healthy, origin xyz=             -0.19              0.0              0.025 rpy=             0.0              0.0             0.0
- added joint kabaong_to_base_link: type fixed, parent base_link, child kabaong, origin xyz=         0.0         -0.075         -0.035 rpy=         0.0          0.0         0.0
- added joint mirror_left_to_kabaong: type fixed, parent kabaong, child mirror_left, origin xyz=             0.375              -0.0555             0.025 rpy=             0.0              0.0             -0.602138592
- added joint mirror_right_to_kabaong: type fixed, parent kabaong, child mirror_right, origin xyz=             0.375              0.0555             0.025 rpy=             0.0              0.0             0.602138592
- joint 1_u_type_robot_waist_bracket_link_to_base_link: origin xyz=         0.0         0.0         0.01905 rpy=         0.0          0.0         0.0 -> xyz=         0.0         0.0         0.01 rpy=         0.0          0.0         0.0

Commit message: Rotate DOF_3 joint by 1.0 radians to create better cartesian paths

File: src/strawberry_picking_rpi_description/urdf/model_for_moveit.urdf (robot description, URDF)
Before this commit: robot strawberry_picking_rpi, 34 links, 33 joints
Joints:
- joint DOF_3: origin xyz=             -0.1055             0.0             0.0 rpy=             0.0             0.0             -1.5707963267948966 -> xyz=             -0.1055             0.0             0.0 rpy=             0.0             0.0             -2.5707963267948966

File: src/strawberry_picking_rpi_description/urdf/strawberry_picking_rpi.urdf.xacro (robot description, xacro)
@@ -262,5 +262,5 @@
             0.0
             0.0
-            ${-pi/2}"
+            ${(-pi/2)-(1.0)}"
             />
             <limit lower="0" upper="${pi}" effort="1000" velocity="${mg996r_velocity_6v}"/>

Commit message: Update moveit config for cameras

File: src/strawberry_picking_rpi_description/urdf/model_for_moveit.urdf (robot description, URDF)
Before this commit: robot strawberry_picking_rpi, 34 links, 33 joints
Links:
- added link depth_camera; visual mesh filename=package://strawberry_picking_rpi_description/meshes/Pi Came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 scale=0.001 0.001 0.001
- added link depth_camera_mount, mass 0.0; collision box size=0.037 0.025 0.11; visual box size=0.037 0.025 0.11
- added link mirror_camera; visual mesh filename=package://strawberry_picking_rpi_description/meshes/Pi Came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 scale=0.001 0.001 0.001
- added link mirror_camera_mount, mass 0.0; collision box size=0.037 0.025 0.062; visual box size=0.037 0.025 0.062
Joints:
- added joint depth_camera_mount_to_kabaong: type fixed, parent kabaong, child depth_camera_mount, origin xyz=             0.07650000000000001             0.0475             0.025 rpy=             0.0              0.0             0.0
- added joint depth_camera_to_depth_camera_mount: type fixed, parent depth_camera_mount, child depth_camera, origin xyz=             0.0             -0.0125             0.09 rpy=             1.5707963267948966             0.0             0.0
- added joint mirror_camera_mount_to_kabaong: type fixed, parent kabaong, child mirror_camera_mount, origin xyz=             0.07650000000000001             0.012499999999999997             0.025 rpy=             0.0              0.0             1.5707963267948966
- added joint mirror_camera_to_mirror_camera_mount: type fixed, parent mirror_camera_mount, child mirror_camera, origin xyz=             0.0             -0.0125             0.041999999999999996 rpy=             1.5707963267948966             0.0             0.0

Commit message: Update URDF

File: src/strawberry_picking_rpi_description/urdf/model_for_moveit.urdf (robot description, URDF)
Before this commit: robot strawberry_picking_rpi, 38 links, 37 joints
Joints:
- joint depth_camera_to_depth_camera_mount: origin xyz=             0.0             -0.0125             0.09 rpy=             1.5707963267948966             0.0             0.0 -> xyz=             0.0             -0.0125             0.09 rpy=             1.5707963267948966             3.141592653589793             0.0
- joint mirror_camera_to_mirror_camera_mount: origin xyz=             0.0             -0.0125             0.041999999999999996 rpy=             1.5707963267948966             0.0             0.0 -> xyz=             0.0             -0.0125             0.041999999999999996 rpy=             1.5707963267948966             3.141592653589793             0.0

File: src/strawberry_picking_rpi_description/urdf/robotic_base_with_accessories.urdf.xacro (robot description, xacro)
@@ -269,5 +269,5 @@
         <link name="mirror_camera">
             <visual>
-                <origin xyz="0.0125 0.0145 0.0" rpy="0.0 0.0 ${pi}"/>
+                <origin xyz="-0.0125 -0.0145 0.0" rpy="0.0 0.0 0.0"/>
                 <geometry>
                     <mesh filename="package://strawberry_picking_rpi_description/meshes/Pi Camera Module v3.STL" scale="0.001 0.001 0.001"/>
@@ -283,5 +283,5 @@
             rpy="
             ${pi/2}
-            0.0
+            ${pi}
             0.0"/>
             <parent link="mirror_camera_mount"/>
@@ -290,5 +290,5 @@
         <link name="depth_camera">
             <visual>
-                <origin xyz="0.0125 0.0145 0.0" rpy="0.0 0.0 ${pi}"/>
+                <origin xyz="-0.0125 -0.0145 0.0" rpy="0.0 0.0 0.0"/>
                 <geometry>
                     <mesh filename="package://strawberry_picking_rpi_description/meshes/Pi Camera Module v3.STL" scale="0.001 0.001 0.001"/>
@@ -304,5 +304,5 @@
             rpy="
             ${pi/2}
-            0.0
+            ${pi}
             0.0"/>
             <parent link="depth_camera_mount"/>
